Commit message: enable simple track visuals

File: urdf/example_track_simple_gazebo.urdf.xacro (robot description, xacro)
@@ -4,5 +4,12 @@
     <xacro:include filename="example_track.urdf.xacro" />
     <!-- -->
-    <xacro:make_track_simple name="track" mass="0.4" length="0.7" radius="0.125" width="0.5" parent="body" sprocket_joint="sprocket_axle" pitch_diameter="0.24" />
+    <xacro:make_track_simple_v name="track" mass="0.4" length="0.7" radius="0.125" width="0.5" parent="body" sprocket_joint="sprocket_axle" pitch_diameter="0.24">
+        <material>
+            <ambient>0.1 0.1 0.1 1</ambient>
+            <diffuse>0.2 0.2 0.2 1</diffuse>
+            <specular>0 0 0 1</specular>
+            <emissive>0 0 0 1</emissive>
+        </material>
+    </xacro:make_track_simple_v>
     <!-- ros_control for gazebo -->
     <gazebo>
