Commit message: use inertial/collision/visual macros

File: urdf/example_track_gazebo.urdf.xacro (robot description, xacro)
@@ -1,4 +1,5 @@
 <robot name="example_track" xmlns:xacro="http://www.ros.org/wiki/xacro">
     <!-- -->
+    <xacro:include filename="$(find gazebo_continuous_track)/urdf/macros_gazebo.urdf.xacro" />
     <xacro:include filename="example_track.urdf.xacro" />
     <!-- -->
@@ -6,12 +7,5 @@
         <link name="upper_segment_link">
             <pose>-0.35 0 0.125 0 0 0</pose>
-            <inertial>
-                <mass>0.1</mass>
-                <inertia>
-                    <ixx>0.01</ixx>
-                    <iyy>0.01</iyy>
-                    <izz>0.01</izz>
-                </inertia>
-            </inertial>
+            <xacro:make_box_inertial pose="0.35 0 0 0 0 0" mass="0.1" size_x="0.7" size_y="0.5" size_z="0.2" />
         </link>
         <joint name="upper_segment_joint" type="prismatic">
@@ -26,12 +20,5 @@
         <link name="front_segment_link">
             <pose>0.35 0 0.125 0 0 0</pose>
-            <inertial>
-                <mass>0.1</mass>
-                <inertia>
-                    <ixx>0.01</ixx>
-                    <iyy>0.01</iyy>
-                    <izz>0.01</izz>
-                </inertia>
-            </inertial>
+            <xacro:make_cylinder_inertial pose="0 0 -0.125 ${pi / 2} 0 0" mass="0.1" length="0.5" radius="0.125" />
         </link>
         <joint name="front_segment_joint" type="revolute">
@@ -46,12 +33,5 @@
         <link name="lower_segment_link">
             <pose>0.35 0 -0.125 0 ${pi} 0</pose>
-            <inertial>
-                <mass>0.1</mass>
-                <inertia>
-                    <ixx>0.01</ixx>
-                    <iyy>0.01</iyy>
-                    <izz>0.01</izz>
-                </inertia>
-            </inertial>
+            <xacro:make_box_inertial pose="0.35 0 0 0 0 0" mass="0.1" size_x="0.7" size_y="0.5" size_z="0.2" />
         </link>
         <joint name="lower_segment_joint" type="prismatic">
@@ -66,12 +46,5 @@
         <link name="rear_segment_link">
             <pose>-0.35 0 -0.125 0 ${pi} 0</pose>
-            <inertial>
-                <mass>0.1</mass>
-                <inertia>
-                    <ixx>0.01</ixx>
-                    <iyy>0.01</iyy>
-                    <izz>0.01</izz>
-                </inertia>
-            </inertial>
+            <xacro:make_cylinder_inertial pose="0 0 -0.125 ${pi / 2} 0 0" mass="0.1" length="0.5" radius="0.125" />
         </link>
         <joint name="rear_segment_joint" type="revolute">
@@ -84,4 +57,12 @@
             </axis>
         </joint>
+        <xacro:property name="element_material">
+            <material>
+                <ambient>0.1 0.1 0.1 1</ambient>
+                <diffuse>0.2 0.2 0.2 1</diffuse>
+                <specular>0 0 0 1</specular>
+                <emissive>0 0 0 1</emissive>
+            </material>
+        </xacro:property>
         <plugin name="continuous_track" filename="libContinuousTrack.so">
             <!-- -->
@@ -111,52 +92,16 @@
             <!-- -->
             <pattern>
-                <elements_per_round>60</elements_per_round>
+                <elements_per_round>80</elements_per_round>
                 <element>
-                    <collision name="collision">
-                        <pose>0 0 0.01 0 0 0</pose>
-                        <geometry>
-                            <box>
-                                <size>0.06 0.2 0.02</size>
-                            </box>
-                        </geometry>
-                    </collision>
-                    <visual name="visual">
-                        <pose>0 0 0.01 0 0 0</pose>
-                        <geometry>
-                            <box>
-                                <size>0.06 0.2 0.02</size>
-                            </box>
-                        </geometry>
-                        <material>
-                            <ambient>0.1 0.1 0.1 1</ambient>
-                            <diffuse>0.2 0.2 0.2 1</diffuse>
-                            <specular>0 0 0 1</specular>
-                            <emissive>0 0 0 1</emissive>
-                        </material>
-                    </visual>
+                    <xacro:make_box_collision pose="0 0 0.01 0 0 0" size="0.05 0.5 0.02" />
+                    <xacro:make_box_visual pose="0 0 0.01 0 0 0" size="0.05 0.5 0.02">
+                        <xacro:insert_block name="element_material" />
+                    </xacro:make_box_visual>
                 </element>
                 <element>
-                    <collision name="collision">
-                        <pose>0 0 0.02 0 0 0</pose>
-                        <geometry>
-                            <box>
-                                <size>0.02 0.2 0.04</size>
-                            </box>
-                        </geometry>
-                    </collision>
-                    <visual name="visual">
-                        <pose>0 0 0.02 0 0 0</pose>
-                        <geometry>
-                            <box>
-                                <size>0.02 0.2 0.04</size>
-                            </box>
-                        </geometry>
-                        <material>
-                            <ambient>0.1 0.1 0.1 1</ambient>
-                            <diffuse>0.2 0.2 0.2 1</diffuse>
-                            <specular>0 0 0 1</specular>
-                            <emissive>0 0 0 1</emissive>
-                        </material>
-                    </visual>
+                    <xacro:make_box_collision pose="0 0 0.02 0 0 0" size="0.02 0.5 0.04" />
+                    <xacro:make_box_visual pose="0 0 0.02 0 0 0" size="0.02 0.5 0.04">
+                        <xacro:insert_block name="element_material" />
+                    </xacro:make_box_visual>
                 </element>
             </pattern>

Commit message: port to latest macros

File: urdf/example_track_gazebo.urdf.xacro (robot description, xacro)
@@ -1,60 +1,12 @@
 <robot name="example_track" xmlns:xacro="http://www.ros.org/wiki/xacro">
     <!-- -->
-    <xacro:include filename="$(find gazebo_continuous_track)/urdf/macros_gazebo.urdf.xacro" />
+    <xacro:include filename="$(find gazebo_continuous_track)/urdf/macros_trajectory_gazebo.urdf.xacro" />
     <xacro:include filename="example_track.urdf.xacro" />
     <!-- -->
+    <xacro:make_straight_segment name_prefix="upper_segment" x="-0.35" z="0.125" mass="0.1" size_x="0.7" size_y="0.5" size_z="0.2" parent="body" />
+    <xacro:make_arc_segment name_prefix="front_segment" x="0.35" z="0.125" mass="0.1" length="0.5" radius="0.125" parent="body" />
+    <xacro:make_straight_segment name_prefix="lower_segment" x="0.35" z="-0.125" pitch="${pi}" mass="0.1" size_x="0.7" size_y="0.5" size_z="0.2" parent="body" />
+    <xacro:make_arc_segment name_prefix="rear_segment" x="-0.35" z="-0.125" pitch="${pi}" mass="0.1" length="0.5" radius="0.125" parent="body" />
     <gazebo>
-        <link name="upper_segment_link">
-            <pose>-0.35 0 0.125 0 0 0</pose>
-            <xacro:make_box_inertial pose="0.35 0 0 0 0 0" mass="0.1" size_x="0.7" size_y="0.5" size_z="0.2" />
-        </link>
-        <joint name="upper_segment_joint" type="prismatic">
-            <pose>0 0 0 0 0 0</pose>
-            <parent>body</parent>
-            <child>upper_segment_link</child>
-            <axis>
-                <xyz>1 0 0</xyz>
-                <use_parent_model_frame>0</use_parent_model_frame>
-            </axis>
-        </joint>
-        <link name="front_segment_link">
-            <pose>0.35 0 0.125 0 0 0</pose>
-            <xacro:make_cylinder_inertial pose="0 0 -0.125 ${pi / 2} 0 0" mass="0.1" length="0.5" radius="0.125" />
-        </link>
-        <joint name="front_segment_joint" type="revolute">
-            <pose>0 0 -0.125 0 0 0</pose>
-            <parent>body</parent>
-            <child>front_segment_link</child>
-            <axis>
-                <xyz>0 1 0</xyz>
-                <use_parent_model_frame>0</use_parent_model_frame>
-            </axis>
-        </joint>
-        <link name="lower_segment_link">
-            <pose>0.35 0 -0.125 0 ${pi} 0</pose>
-            <xacro:make_box_inertial pose="0.35 0 0 0 0 0" mass="0.1" size_x="0.7" size_y="0.5" size_z="0.2" />
-        </link>
-        <joint name="lower_segment_joint" type="prismatic">
-            <pose>0 0 0 0 0 0</pose>
-            <parent>body</parent>
-            <child>lower_segment_link</child>
-            <axis>
-                <xyz>1 0 0</xyz>
-                <use_parent_model_frame>0</use_parent_model_frame>
-            </axis>
-        </joint>
-        <link name="rear_segment_link">
-            <pose>-0.35 0 -0.125 0 ${pi} 0</pose>
-            <xacro:make_cylinder_inertial pose="0 0 -0.125 ${pi / 2} 0 0" mass="0.1" length="0.5" radius="0.125" />
-        </link>
-        <joint name="rear_segment_joint" type="revolute">
-            <pose>0 0 -0.125 0 0 0</pose>
-            <parent>body</parent>
-            <child>rear_segment_link</child>
-            <axis>
-                <xyz>0 1 0</xyz>
-                <use_parent_model_frame>0</use_parent_model_frame>
-            </axis>
-        </joint>
         <xacro:property name="element_material">
             <material>

File: urdf/example_track_simple_gazebo.urdf.xacro (robot description, xacro)
@@ -2,6 +2,5 @@
     <!-- -->
     <xacro:include filename="example_track.urdf.xacro" />
-    <!-- -->
-    <xacro:include filename="$(find gazebo_continuous_track)/urdf/macros_gazebo.urdf.xacro" />
+    <xacro:include filename="$(find gazebo_continuous_track)/urdf/macros_populate_gazebo.urdf.xacro" />
     <!-- -->
     <xacro:populate_wheels name_prefix="track_wheel" x="0.35" dx="-0.70" dpitch="${pi}" mass="0.1" length="0.2" radius="0.125" count="2" />

Commit message: use make_track* macros

File: urdf/example_track_gazebo.urdf.xacro (robot description, xacro)
@@ -1,63 +1,34 @@
 <robot name="example_track" xmlns:xacro="http://www.ros.org/wiki/xacro">
     <!-- -->
-    <xacro:include filename="$(find gazebo_continuous_track)/urdf/macros_trajectory_gazebo.urdf.xacro" />
+    <xacro:include filename="$(find gazebo_continuous_track)/urdf/macros_track_gazebo.urdf.xacro" />
     <xacro:include filename="example_track.urdf.xacro" />
     <!-- -->
-    <xacro:make_straight_segment name_prefix="upper_segment" x="-0.35" z="0.125" mass="0.1" size_x="0.7" size_y="0.5" size_z="0.2" parent="body" />
-    <xacro:make_arc_segment name_prefix="front_segment" x="0.35" z="0.125" mass="0.1" length="0.5" radius="0.125" parent="body" />
-    <xacro:make_straight_segment name_prefix="lower_segment" x="0.35" z="-0.125" pitch="${pi}" mass="0.1" size_x="0.7" size_y="0.5" size_z="0.2" parent="body" />
-    <xacro:make_arc_segment name_prefix="rear_segment" x="-0.35" z="-0.125" pitch="${pi}" mass="0.1" length="0.5" radius="0.125" parent="body" />
+    <xacro:property name="element_material">
+        <material>
+            <ambient>0.1 0.1 0.1 1</ambient>
+            <diffuse>0.2 0.2 0.2 1</diffuse>
+            <specular>0 0 0 1</specular>
+            <emissive>0 0 0 1</emissive>
+        </material>
+    </xacro:property>
+    <xacro:make_track name="track" mass="0.4" length="0.7" radius="0.125" width="0.5" parent="body" sprocket="sprocket_axle" pitch_diameter="0.24">
+        <pattern>
+            <elements_per_round>80</elements_per_round>
+            <element>
+                <xacro:make_box_collision pose="0 0 0.01 0 0 0" size="0.05 0.5 0.02" />
+                <xacro:make_box_visual pose="0 0 0.01 0 0 0" size="0.05 0.5 0.02">
+                    <xacro:insert_block name="element_material" />
+                </xacro:make_box_visual>
+            </element>
+            <element>
+                <xacro:make_box_collision pose="0 0 0.02 0 0 0" size="0.02 0.5 0.04" />
+                <xacro:make_box_visual pose="0 0 0.02 0 0 0" size="0.02 0.5 0.04">
+                    <xacro:insert_block name="element_material" />
+                </xacro:make_box_visual>
+            </element>
+        </pattern>
+    </xacro:make_track>
+    <!-- ros_control for gazebo -->
     <gazebo>
-        <xacro:property name="element_material">
-            <material>
-                <ambient>0.1 0.1 0.1 1</ambient>
-                <diffuse>0.2 0.2 0.2 1</diffuse>
-                <specular>0 0 0 1</specular>
-                <emissive>0 0 0 1</emissive>
-            </material>
-        </xacro:property>
-        <plugin name="continuous_track" filename="libContinuousTrack.so">
-            <!-- -->
-            <sprocket>
-                <joint>sprocket_axle</joint>
-                <pitch_diameter>0.24</pitch_diameter>
-            </sprocket>
-            <!-- -->
-            <trajectory>
-                <segment>
-                    <joint>upper_segment_joint</joint>
-                    <end_position>0.7</end_position>
-                </segment>
-                <segment>
-                    <joint>front_segment_joint</joint>
-                    <end_position>${pi}</end_position>
-                </segment>
-                <segment>
-                    <joint>lower_segment_joint</joint>
-                    <end_position>0.7</end_position>
-                </segment>
-                <segment>
-                    <joint>rear_segment_joint</joint>
-                    <end_position>${pi}</end_position>
-                </segment>
-            </trajectory>
-            <!-- -->
-            <pattern>
-                <elements_per_round>80</elements_per_round>
-                <element>
-                    <xacro:make_box_collision pose="0 0 0.01 0 0 0" size="0.05 0.5 0.02" />
-                    <xacro:make_box_visual pose="0 0 0.01 0 0 0" size="0.05 0.5 0.02">
-                        <xacro:insert_block name="element_material" />
-                    </xacro:make_box_visual>
-                </element>
-                <element>
-                    <xacro:make_box_collision pose="0 0 0.02 0 0 0" size="0.02 0.5 0.04" />
-                    <xacro:make_box_visual pose="0 0 0.02 0 0 0" size="0.02 0.5 0.04">
-                        <xacro:insert_block name="element_material" />
-                    </xacro:make_box_visual>
-                </element>
-            </pattern>
-        </plugin>
-        <!-- ros_control for gazebo -->
         <plugin name="gazebo_ros_control" filename="libgazebo_ros_control.so">
             <robotSimType>gazebo_ros_control/DefaultRobotHWSim</robotSimType>

File: urdf/example_track_simple_gazebo.urdf.xacro (robot description, xacro)
@@ -1,37 +1,10 @@
 <robot name="example_track_simple" xmlns:xacro="http://www.ros.org/wiki/xacro">
     <!-- -->
+    <xacro:include filename="$(find gazebo_continuous_track)/urdf/macros_track_simple_gazebo.urdf.xacro" />
     <xacro:include filename="example_track.urdf.xacro" />
-    <xacro:include filename="$(find gazebo_continuous_track)/urdf/macros_populate_gazebo.urdf.xacro" />
     <!-- -->
-    <xacro:populate_wheels name_prefix="track_wheel" x="0.35" dx="-0.70" dpitch="${pi}" mass="0.1" length="0.2" radius="0.125" count="2" />
-    <xacro:populate_axles name_prefix="track_axle" parent="body" child_prefix="track_wheel" count="2"/>
-    <xacro:populate_boards name_prefix="track_board" z="0.12" dz="-0.24" dpitch="${pi}" mass="0.1" size_x="0.7" size_y="0.2" size_z="0.01" count="2" />
-    <xacro:populate_sliders name_prefix="track_slider" parent="body" child_prefix="track_board" count="2"/>
+    <xacro:make_track_simple name="track" mass="0.4" length="0.7" radius="0.125" width="0.2" parent="body" sprocket="sprocket_axle" pitch_diameter="0.24" />
+    <!-- ros_control for gazebo -->
     <gazebo>
-        <plugin name="continuous_track_simple" filename="libContinuousTrackSimple.so">
-            <!-- -->
-            <sprocket>
-                <joint>sprocket_axle</joint>
-                <pitch_diameter>0.24</pitch_diameter>
-            </sprocket>
-            <!-- -->
-            <track>
-                <segment>
-                    <joint>track_slider1</joint>
-                </segment>
-                <segment>
-                    <joint>track_axle1</joint>
-                    <pitch_diameter>0.24</pitch_diameter>
-                </segment>
-                <segment>
-                    <joint>track_slider2</joint>
-                </segment>
-                <segment>
-                    <joint>track_axle2</joint>
-                    <pitch_diameter>0.24</pitch_diameter>
-                </segment>
-            </track>
-        </plugin>
-        <!-- ros_control for gazebo -->
         <plugin name="gazebo_ros_control" filename="libgazebo_ros_control.so">
             <robotSimType>gazebo_ros_control/DefaultRobotHWSim</robotSimType>

Commit message: update for latest macros

File: urdf/example_track_gazebo.urdf.xacro (robot description, xacro)
@@ -4,5 +4,5 @@
     <xacro:include filename="example_track.urdf.xacro" />
     <!-- -->
-    <xacro:property name="element_material">
+    <xacro:property name="track_material">
         <material>
             <ambient>0.1 0.1 0.1 1</ambient>
@@ -12,15 +12,11 @@
         </material>
     </xacro:property>
-    <xacro:make_track name="track" mass="0.4" length="0.7" radius="0.125" width="0.5" parent="body" sprocket_joint="sprocket_axle" pitch_diameter="0.24">
+    <xacro:make_track name="track" mass="0.4" length="0.7" radius="0.115" width="0.5" parent="body" sprocket_joint="sprocket_axle" pitch_diameter="0.24">
+        <xacro:insert_block name="track_material" />
         <pattern>
-            <elements_per_round>80</elements_per_round>
+            <elements_per_round>40</elements_per_round>
             <element>
-                <xacro:make_box_element pose="0 0 -0.02 0 0 0" size="0.035 0.5 0.02">
-                    <xacro:insert_block name="element_material" />
-                </xacro:make_box_element>
-            </element>
-            <element>
-                <xacro:make_box_element pose="0 0 -0.015 0 0 0" size="0.02 0.5 0.03">
-                    <xacro:insert_block name="element_material" />
+                <xacro:make_box_element pose="0 0 0 0 0 0" size="0.02 0.5 0.02">
+                    <xacro:insert_block name="track_material" />
                 </xacro:make_box_element>
             </element>
