Commit message: reasonable inertia

File: urdf/example_track.urdf.xacro (robot description, xacro)
@@ -6,9 +6,25 @@
     <!--     * an axle and actuator for the sprocket                                 -->
     <!-- Other entities specialized for Gazebo are defined in example_gazebo.urdf .  -->
+    <xacro:macro name="make_body_inertia" params="mass size_x size_y size_z">
+        <inertial>
+            <mass value="${mass}" />
+            <inertia
+                ixx="${mass * (size_y * size_y + size_z * size_z) / 12}" ixy="0" ixz="0"
+                iyy="${mass * (size_z * size_z + size_x * size_x) / 12}" iyz="0"
+                izz="${mass * (size_x * size_x + size_y * size_y) / 12}" />
+        </inertial>
+    </xacro:macro>
+    <xacro:macro name="make_sprocket_inertia" params="mass radius length">
+        <inertial>
+            <mass value="${mass}" />
+            <!-- assuming axis of cylinder is y, not z -->
+            <inertia
+                ixx="${mass * (radius * radius / 4 + length * length / 12)}" ixy="0" ixz="0"
+                iyy="${mass * radius * radius / 2}" iyz="0"
+                izz="${mass * (radius * radius / 4 + length * length / 12)}" />
+        </inertial>
+    </xacro:macro>
     <link name="body">
-        <inertial>
-            <mass value="1" />
-            <inertia ixx="0.1" ixy="0" ixz="0" iyy="0.1" iyz="0" izz="0.1" />
-        </inertial>
+        <xacro:make_body_inertia mass="1" size_x="0.5" size_y="0.2" size_z="0.2" />
         <visual>
             <geometry>
@@ -26,8 +42,5 @@
     </link>
     <link name="sprocket">
-        <inertial>
-            <mass value="0.2" />
-            <inertia ixx="0.01" ixy="0" ixz="0" iyy="0.01" iyz="0" izz="0.01" />
-        </inertial>
+        <xacro:make_sprocket_inertia mass="0.2" radius="0.1" length="0.2" />
         <visual>
             <origin xyz="0 0 0" rpy="${pi / 2} 0 0" />

Commit message: change track width to 0.5

File: urdf/example_track.urdf.xacro (robot description, xacro)
@@ -26,8 +26,8 @@
     </xacro:macro>
     <link name="body">
-        <xacro:make_body_inertia mass="1" size_x="0.5" size_y="0.2" size_z="0.2" />
+        <xacro:make_body_inertia mass="1" size_x="0.5" size_y="0.5" size_z="0.2" />
         <visual>
             <geometry>
-                <box size="0.5 0.2 0.2" />
+                <box size="0.5 0.5 0.2" />
             </geometry>
             <material name="red">
@@ -37,14 +37,14 @@
         <collision>
             <geometry>
-                <box size="0.5 0.2 0.2" />
+                <box size="0.5 0.5 0.2" />
             </geometry>
         </collision>
     </link>
     <link name="sprocket">
-        <xacro:make_sprocket_inertia mass="0.2" radius="0.1" length="0.2" />
+        <xacro:make_sprocket_inertia mass="0.2" radius="0.1" length="0.5" />
         <visual>
             <origin xyz="0 0 0" rpy="${pi / 2} 0 0" />
             <geometry>
-                <cylinder radius="0.1" length="0.2" />
+                <cylinder radius="0.1" length="0.5" />
             </geometry>
             <material name="grey">
@@ -55,10 +55,10 @@
             <origin xyz="0 0 0" rpy="${pi / 2} 0 0" />
             <geometry>
-                <cylinder radius="0.1" length="0.2" />
+                <cylinder radius="0.1" length="0.5" />
             </geometry>
         </collision>
     </link>
     <joint name="sprocket_axle" type="continuous">
-        <origin xyz="0.35 0 0" rpy="0 0 0" />
+        <origin xyz="0.375 0 0" rpy="0 0 0" />
         <parent link="body" />
         <child link="sprocket" />

File: urdf/example_track_simple_gazebo.urdf.xacro (robot description, xacro)
@@ -4,5 +4,5 @@
     <xacro:include filename="example_track.urdf.xacro" />
     <!-- -->
-    <xacro:make_track_simple name="track" mass="0.4" length="0.7" radius="0.125" width="0.2" parent="body" sprocket_joint="sprocket_axle" pitch_diameter="0.24" />
+    <xacro:make_track_simple name="track" mass="0.4" length="0.7" radius="0.125" width="0.5" parent="body" sprocket_joint="sprocket_axle" pitch_diameter="0.24" />
     <!-- ros_control for gazebo -->
     <gazebo>

Commit message: edit size of track body for better looking

File: urdf/example_track.urdf.xacro (robot description, xacro)
@@ -26,8 +26,8 @@
     </xacro:macro>
     <link name="body">
-        <xacro:make_body_inertia mass="1" size_x="0.5" size_y="0.5" size_z="0.2" />
+        <xacro:make_body_inertia mass="1" size_x="0.5" size_y="0.51" size_z="0.2" />
         <visual>
             <geometry>
-                <box size="0.5 0.5 0.2" />
+                <box size="0.5 0.51 0.2" />
             </geometry>
             <material name="red">
@@ -37,14 +37,14 @@
         <collision>
             <geometry>
-                <box size="0.5 0.5 0.2" />
+                <box size="0.51 0.5 0.2" />
             </geometry>
         </collision>
     </link>
     <link name="sprocket">
-        <xacro:make_sprocket_inertia mass="0.2" radius="0.1" length="0.5" />
+        <xacro:make_sprocket_inertia mass="0.2" radius="0.1" length="0.51" />
         <visual>
             <origin xyz="0 0 0" rpy="${pi / 2} 0 0" />
             <geometry>
-                <cylinder radius="0.1" length="0.5" />
+                <cylinder radius="0.1" length="0.51" />
             </geometry>
             <material name="grey">
@@ -55,10 +55,10 @@
             <origin xyz="0 0 0" rpy="${pi / 2} 0 0" />
             <geometry>
-                <cylinder radius="0.1" length="0.5" />
+                <cylinder radius="0.1" length="0.51" />
             </geometry>
         </collision>
     </link>
     <joint name="sprocket_axle" type="continuous">
-        <origin xyz="0.375 0 0" rpy="0 0 0" />
+        <origin xyz="0.35 0 0" rpy="0 0 0" />
         <parent link="body" />
         <child link="sprocket" />

Commit message: add an idler wheel

File: urdf/example_track.urdf.xacro (robot description, xacro)
@@ -5,26 +5,22 @@
     <!--     * a sprocket to drive the track                                         -->
     <!--     * an axle and actuator for the sprocket                                 -->
+    <!--     * an idler wheel on the other side of the sprocket                      -->
     <!-- Other entities specialized for Gazebo are defined in example_gazebo.urdf .  -->
-    <xacro:macro name="make_body_inertia" params="mass size_x size_y size_z">
+    <xacro:macro name="make_box_inertia" params="mass size_x size_y size_z">
         <inertial>
             <mass value="${mass}" />
-            <inertia
-                ixx="${mass * (size_y * size_y + size_z * size_z) / 12}" ixy="0" ixz="0"
-                iyy="${mass * (size_z * size_z + size_x * size_x) / 12}" iyz="0"
-                izz="${mass * (size_x * size_x + size_y * size_y) / 12}" />
+            <inertia ixx="${mass * (size_y * size_y + size_z * size_z) / 12}" ixy="0" ixz="0" iyy="${mass * (size_z * size_z + size_x * size_x) / 12}" iyz="0" izz="${mass * (size_x * size_x + size_y * size_y) / 12}" />
         </inertial>
     </xacro:macro>
-    <xacro:macro name="make_sprocket_inertia" params="mass radius length">
+    <xacro:macro name="make_wheel_inertia" params="mass radius length">
         <inertial>
             <mass value="${mass}" />
             <!-- assuming axis of cylinder is y, not z -->
-            <inertia
-                ixx="${mass * (radius * radius / 4 + length * length / 12)}" ixy="0" ixz="0"
-                iyy="${mass * radius * radius / 2}" iyz="0"
-                izz="${mass * (radius * radius / 4 + length * length / 12)}" />
+            <inertia ixx="${mass * (radius * radius / 4 + length * length / 12)}" ixy="0" ixz="0" iyy="${mass * radius * radius / 2}" iyz="0" izz="${mass * (radius * radius / 4 + length * length / 12)}" />
         </inertial>
     </xacro:macro>
+    <!-- body to be wrapped by the track -->
     <link name="body">
-        <xacro:make_body_inertia mass="1" size_x="0.5" size_y="0.51" size_z="0.2" />
+        <xacro:make_box_inertia mass="1" size_x="0.5" size_y="0.51" size_z="0.2" />
         <visual>
             <geometry>
@@ -41,6 +37,7 @@
         </collision>
     </link>
+    <!-- sprocket driving the track -->
     <link name="sprocket">
-        <xacro:make_sprocket_inertia mass="0.2" radius="0.1" length="0.51" />
+        <xacro:make_wheel_inertia mass="0.2" radius="0.1" length="0.51" />
         <visual>
             <origin xyz="0 0 0" rpy="${pi / 2} 0 0" />
@@ -74,3 +71,27 @@
         </actuator>
     </transmission>
+    <!-- idler on the other side of the sprocket -->
+    <link name="idler">
+        <xacro:make_wheel_inertia mass="0.2" radius="0.1" length="0.51" />
+        <visual>
+            <origin xyz="0 0 0" rpy="${pi / 2} 0 0" />
+            <geometry>
+                <cylinder radius="0.1" length="0.51" />
+            </geometry>
+            <material name="grey">
+                <color rgba="0.5 0.5 0.5 1.0" />
+            </material>
+        </visual>
+        <collision>
+            <origin xyz="0 0 0" rpy="${pi / 2} 0 0" />
+            <geometry>
+                <cylinder radius="0.1" length="0.51" />
+            </geometry>
+        </collision>
+    </link>
+    <joint name="idler_axle" type="fixed">
+        <origin xyz="-0.35 0 0" rpy="0 0 0" />
+        <parent link="body" />
+        <child link="idler" />
+    </joint>
 </robot>

Commit message: add teeth of sprocket to visualize rotation

File: urdf/example_track.urdf.xacro (robot description, xacro)
@@ -43,9 +43,21 @@
             <origin xyz="0 0 0" rpy="${pi / 2} 0 0" />
             <geometry>
-                <cylinder radius="0.1" length="0.51" />
+                <cylinder radius="0.08" length="0.51" />
             </geometry>
             <material name="grey">
                 <color rgba="0.5 0.5 0.5 1.0" />
             </material>
+        </visual>
+        <visual>
+            <geometry>
+                <box size="0.01 0.51 0.20" />
+            </geometry>
+            <material name="grey" />
+        </visual>
+        <visual>
+            <geometry>
+                <box size="0.20 0.51 0.01" />
+            </geometry>
+            <material name="grey" />
         </visual>
         <collision>
@@ -79,7 +91,5 @@
                 <cylinder radius="0.1" length="0.51" />
             </geometry>
-            <material name="grey">
-                <color rgba="0.5 0.5 0.5 1.0" />
-            </material>
+            <material name="grey" />
         </visual>
         <collision>

Commit message: change sprocket & idler radius for better looking

File: urdf/example_track.urdf.xacro (robot description, xacro)
@@ -39,5 +39,5 @@
     <!-- sprocket driving the track -->
     <link name="sprocket">
-        <xacro:make_wheel_inertia mass="0.2" radius="0.1" length="0.51" />
+        <xacro:make_wheel_inertia mass="0.2" radius="0.08" length="0.51" />
         <visual>
             <origin xyz="0 0 0" rpy="${pi / 2} 0 0" />
@@ -64,5 +64,5 @@
             <origin xyz="0 0 0" rpy="${pi / 2} 0 0" />
             <geometry>
-                <cylinder radius="0.1" length="0.51" />
+                <cylinder radius="0.08" length="0.51" />
             </geometry>
         </collision>
@@ -85,9 +85,9 @@
     <!-- idler on the other side of the sprocket -->
     <link name="idler">
-        <xacro:make_wheel_inertia mass="0.2" radius="0.1" length="0.51" />
+        <xacro:make_wheel_inertia mass="0.2" radius="0.08" length="0.51" />
         <visual>
             <origin xyz="0 0 0" rpy="${pi / 2} 0 0" />
             <geometry>
-                <cylinder radius="0.1" length="0.51" />
+                <cylinder radius="0.08" length="0.51" />
             </geometry>
             <material name="grey" />
@@ -96,5 +96,5 @@
             <origin xyz="0 0 0" rpy="${pi / 2} 0 0" />
             <geometry>
-                <cylinder radius="0.1" length="0.51" />
+                <cylinder radius="0.08" length="0.51" />
             </geometry>
         </collision>

Commit message: remove material settings for ROS, which are not used for gazebo

File: urdf/example_track.urdf.xacro (robot description, xacro)
@@ -27,7 +27,4 @@
                 <box size="0.5 0.51 0.2" />
             </geometry>
-            <material name="red">
-                <color rgba="0.7 0.0 0.0 1.0" />
-            </material>
         </visual>
         <collision>
@@ -45,7 +42,4 @@
                 <cylinder radius="0.08" length="0.51" />
             </geometry>
-            <material name="grey">
-                <color rgba="0.5 0.5 0.5 1.0" />
-            </material>
         </visual>
         <visual>
@@ -53,5 +47,4 @@
                 <box size="0.01 0.51 0.20" />
             </geometry>
-            <material name="grey" />
         </visual>
         <visual>
@@ -59,5 +52,4 @@
                 <box size="0.20 0.51 0.01" />
             </geometry>
-            <material name="grey" />
         </visual>
         <collision>
@@ -91,5 +83,4 @@
                 <cylinder radius="0.08" length="0.51" />
             </geometry>
-            <material name="grey" />
         </visual>
         <collision>
